File: hardware/SOA-driver.kicad_sch (KiCad schematic)
At the start: 3 parts, among them J1 BASYS3, U1 MCP4728

Commit message: feat: added firmware and better dir management, updates gitignore for vivado files
Other:
- title: Laser Diode Driver -> SOA Driver Board
Changed lines of the file:
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@@
 	(paper "A4")
 	(title_block
-		(title "Laser Diode Driver")
+		(title "SOA Driver Board")
 		(date "2024-03-27")
 		(comment 1 "Mirco Tollardo")
@@
 		)
 		(instances
-			(project "LD-Driver"
+			(project "SOA-driver"
 				(path "/aef12ca3-3d60-44eb-99b6-8bdd18a4b35c"
 					(page "2")
@@
 		)
 		(instances
-			(project "LD-Driver"
+			(project "SOA-driver"
 				(path "/aef12ca3-3d60-44eb-99b6-8bdd18a4b35c"
 					(page "3")

Commit message: fix: tidier schematic
Parts:
- removed C1: 100n, Capacitor_SMD:C_0603_1608Metric, symbol Device:C
- removed J1: BASYS3, Connector_PinHeader_2.54mm:PinHeader_2x07_P2.54mm_Horizontal, symbol Connector_Generic:Conn_02x07_Odd_Even
- removed U1: MCP4728, Package_SO:MSOP-10_3x3mm_P0.5mm, symbol Analog_DAC:MCP4728
Other:
- sheet Driver renamed SOA Driver
- sheet Power renamed 5V DCDC converter
- added sheet From Basys3 (external.kicad_sch)
- added sheet TEC controller (tec-controller.kicad_sch)
- sheet SOA Driver ports: added none; removed CTRL_H_DAC, CTRL_L_DAC, CTRL_SELECT, ILD_MON, ITEC_MON, LD_EN, LD_MODULATION, OVERTMP_ALM, TEC_TEMPSETPOINT_DAC, TEC_VMAX_DAC, TEC_~{SHD}, UNDERTMP_ALM
