File: hardware/SOA-driver.kicad_pcb (KiCad board)
At the start: 2 copper layers, 107.5 x 72 mm, 134 parts, among them J1 BASYS3, J2 BUTTERFLY, J3 Barrel_Jack_Switch, J4 SELECTOR, J5 SELECTOR_2, J6 5V EXT, Q1 RJK0355DSP, Q10 RJK0355DSP, Q2 RJK0355DSP, Q3 SiRC18DP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

Commit message: feat: decent readme as user manual
Parts:
- added R28: 10, Resistor_SMD:R_0603_1608Metric, B.Cu at (135.9, 60.8)
- added R29: 1k, Resistor_SMD:R_0603_1608Metric, B.Cu at (139.0, 62.0)
- J1: footprint Connector_PinHeader_2.54mm:PinHeader_2x07_P2.54mm_Horizontal -> Connector_PinHeader_2.54mm:PinHeader_2x07_P2.54mm_Vertical
- moved C1 1.17 mm to (132.6, 60.8)
- moved J1 0.11 mm to (135.9, 58.5)
Connections:
- net /Driver/1V5ADC renamed /TEC controller/1V5ADC
- net /Driver/BFB- renamed /TEC controller/BFB-
- net /Driver/CTRL_H_DAC renamed CTRL_H_DAC
- net /Driver/CTRL_L_DAC renamed CTRL_L_DAC
- net /Driver/FB+ renamed /TEC controller/TTEC_SETPOINT_DAC
- net /Driver/INT- renamed /TEC controller/INT-
- net /Driver/INTOUT renamed /TEC controller/INTOUT
- net /Driver/LD renamed /SOA Driver/LD
- net /Driver/MAXV_DAC renamed /TEC controller/MAXV_DAC
- net /Driver/NTC+ renamed /SOA Driver/NTC+
- net /Driver/PWMGH renamed /SOA Driver/PWMGH
- net /Driver/PWMGL renamed /SOA Driver/PWMGL
- net /Driver/Pin_1 renamed /SOA Driver/Pin_1
- net /Driver/Pin_10 renamed /SOA Driver/Pin_10
- net /Driver/Pin_11 renamed /SOA Driver/Pin_11
- net /Driver/Pin_12 renamed /SOA Driver/Pin_12
- net /Driver/Pin_13 renamed /SOA Driver/Pin_13
- net /Driver/Pin_14 renamed /SOA Driver/Pin_14
- net /Driver/Pin_2 renamed /SOA Driver/Pin_2
- net /Driver/Pin_3 renamed /SOA Driver/Pin_3
- net /Driver/Pin_4 renamed /SOA Driver/Pin_4
- net /Driver/Pin_5 renamed /SOA Driver/Pin_5
- net /Driver/Pin_6 renamed /SOA Driver/Pin_6
- net /Driver/Pin_7 renamed /SOA Driver/Pin_7
- net /Driver/Pin_8 renamed /SOA Driver/Pin_8
- net /Driver/Pin_9 renamed /SOA Driver/Pin_9
- net /Driver/SENSE+ renamed /SOA Driver/SENSE+
- net /Driver/SENSE- renamed /SOA Driver/SENSE-
- net /Driver/SW renamed /SOA Driver/SW
- net /Driver/TEC+ renamed /SOA Driver/TEC+
- net /Driver/TEC- renamed /SOA Driver/TEC-
- net /ILD_MON renamed ILD_MON
- net /ITEC_MON renamed ITEC_MON
- net /LD_EN renamed LD_EN
- net /OVERTMP_ALM renamed OVERTMP_ALM
- net /Power/DH renamed /5V DCDC converter/DH
- net /Power/DL renamed /5V DCDC converter/DL
- net /Power/FB renamed /5V DCDC converter/FB
- net /RDY/~{BSY} renamed RDY/~{BSY}
- net /SCL renamed SCL
- net /SDA renamed SDA
- net /UNDERTMP_ALM renamed UNDERTMP_ALM
- net /~{LDAC} renamed ~{LDAC}
- C42 pad 1: Net-(U5-VDD) -> Net-(D3-A)
- J1 pad 13: /TEC_EN -> TEC_EN
- J1 pad 2: /LD_MOD -> LD_MOD
- J1 pad 4: /CTRL_SEL -> CTRL_SEL
- J4 pad 11: GNDA -> /SOA Driver/NTC-
- R4 pad 2: /TEC_EN -> TEC_~{SHD}
- TP7 pad 1: /LD_MOD -> LD_MODULATION
- U2 pad 19: /CTRL_SEL -> CTRL_SELECT
- U2 pad 20: /LD_MOD -> LD_MODULATION
- U3 pad 11: /TEC_EN -> TEC_~{SHD}
- U5 pad 1: Net-(U5-VDD) -> Net-(D3-A)
Routing:
- net TEC_EN: track 0.00 -> 74.9 mm, vias 0 -> 4
- net /TEC_EN: track 74.9 -> 0.00 mm, vias 4 -> 0
- net LD_MODULATION: track 0.00 -> 55.5 mm, vias 0 -> 3
- net /LD_MOD: track 55.5 -> 0.00 mm, vias 3 -> 0
- net /CTRL_SEL: track 53.1 -> 0.00 mm, vias 3 -> 0
- net CTRL_SELECT: track 0.00 -> 53.1 mm, vias 0 -> 3
- net +3V3: track 36.0 -> 42.3 mm
- net Net-(U5-VDD): track 4.85 -> 0.00 mm
- net Net-(D3-A): track 3.70 -> 8.55 mm
- net SCL: track 6.12 -> 10.2 mm
- net SDA: track 9.13 -> 10.3 mm
- net ILD_MON: track 35.4 -> 36.5 mm
Other:
- board text added: "1"
- board text added: "14"
- board text added: "7"
- board text added: "8"
